File: ioboard-panel-minimoog.kicad_pcb (KiCad board)
At the start: 2 copper layers, 50.5 x 128.5 mm, 5 parts

Commit message: fix
Other:
- board text added: "jlcjlcjlcjlcjlcjlcjlcjlcjlcjlcjlcjlcjlcjlc"
Changed lines of the file:
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@@
 		(layer "Edge.Cuts")
+	)
+	(gr_text "jlcjlcjlcjlcjlcjlcjlcjlcjlcjlcjlcjlcjlcjlc"
+		(at 129.2511 110.3111 0)
+		(layer "B.SilkS")
+		(effects
+			(font
+				(size 1.5 1.5)
+				(thickness 0.3)
+				(bold yes)
+			)
+			(justify left bottom)
+		)
 	)
 	(gr_text "YUSynth\nMiniMoog VCF\nby Gerbster\nIOboard redesign+panel\nby Borgar"
