File: ioboard.kicad_pcb (KiCad board)
At the start: 2 copper layers, 42.2 x 99.7 mm, 19 parts

Commit message: pics
Routing:
- net (no net): vias 1 -> 0
Other:
- board size 42.2 x 99.7 mm -> 41.9 x 99.7 mm
Changed lines of the file:
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@@
 		(pad_to_mask_clearance 0)
 		(allow_soldermask_bridges_in_footprints no)
-		(grid_origin 148.5011 57.0611)
+		(grid_origin 169.2061 154.862529)
 		(pcbplotparams
 			(layerselection 0x00010fc_ffffffff)
@@
 		(layer "Cmts.User")
 	)
-	(gr_line
-		(start 127.2961 154.8511)
-		(end 169.2061 154.8511)
-		(stroke
-			(width 0.05)
-			(type solid)
-		)
-		(layer "Edge.Cuts")
-	)
-	(gr_line
-		(start 169.2061 55.1561)
-		(end 169.2061 100.8761)
-		(stroke
-			(width 0.05)
-			(type solid)
-		)
-		(layer "Edge.Cuts")
-	)
-	(gr_line
-		(start 127.2961 154.8511)
-		(end 127.2961 55.1561)
-		(stroke
-			(width 0.05)
-			(type solid)
-		)
-		(layer "Edge.Cuts")
-	)
-	(gr_line
-		(start 169.2061 55.1561)
-		(end 127.2961 55.1561)
-		(stroke
-			(width 0.05)
-			(type solid)
-		)
-		(layer "Edge.Cuts")
-	)
-	(gr_line
-		(start 169.4561 154.8511)
-		(end 169.4561 70.3961)
+	(gr_rect
+		(start 127.28365 55.1561)
+		(end 169.2061 154.862529)
 		(stroke
 			(width 0.05)
-			(type solid)
+			(type default)
 		)
+		(fill none)
 		(layer "Edge.Cuts")
 	)
@@
 		(layer "Dwgs.User")
 		(pts
+			(xy 127.3429 155.0543) (xy 127.2961 55.1561)
+		)
+		(height -12.827558)
+		(gr_text "99.8982 mm"
+			(at 115.641943 105.11067 -89.97315825)
+			(layer "Dwgs.User")
+			(effects
+				(font
+					(size 1 1)
+					(thickness 0.15)
+				)
+			)
+		)
+		(format
+			(prefix "")
+			(suffix "")
+			(units 3)
+			(units_format 1)
+			(precision 4)
+		)
+		(style
+			(thickness 0.1)
+			(arrow_length 1.27)
+			(text_position_mode 0)
+			(extension_height 0.58642)
+			(extension_offset 0.5) keep_text_aligned)
+	)
+	(dimension
+		(type aligned)
+		(layer "Dwgs.User")
+		(pts
 			(xy 127.3411 55.1561) (xy 169.2511 55.1561)
 		)
@@
 			(extension_offset 0.5) keep_text_aligned)
 	)
-	(via
-		(at 186.5011 67.0611)
-		(size 0.6)
-		(drill 0.3)
-		(layers "F.Cu" "B.Cu")
-		(net 0)
-	)
 	(segment
 		(start 167.551408 70.409411)
@@
 		(polygon
 			(pts
-				(xy 169.6593 155.0543) (xy 127.3429 155.0543) (xy 127.3429 54.9529) (xy 169.6593 54.9529)
+				(xy 169.2061 154.8511) (xy 127.2961 154.8511) (xy 127.2961 55.1561) (xy 169.2061 55.1561)
 			)
 		)
@@
 		(polygon
 			(pts
-				(xy 169.6593 155.0543) (xy 127.3429 155.0543) (xy 127.3429 54.9529) (xy 169.6593 54.9529)
+				(xy 169.2061 154.862529) (xy 127.2961 154.8511) (xy 127.2961 55.1561) (xy 169.2061 55.1561)
 			)
 		)

Commit message: asd
Parts:
- R33, R34: value 100k -> 150k
Changed lines of the file:
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@@
 			)
 		)
-		(property "Value" "100k"
+		(property "Value" "150k"
 			(at -1.6256 0.4826 0)
 			(unlocked yes)
@@
 			)
 		)
-		(property "Value" "100k"
+		(property "Value" "150k"
 			(at -1.81 0.5 -90)
 			(unlocked yes)
